File: FinalTree.kicad_sch (KiCad schematic)
At the start: 8 parts, among them U34 74LS283, U35 74LS283, U36 74LS283, U37 74LS283

Commit message: Fixed ERC issues and applied Footprints
Parts:
- C34, C35, C36, C37: footprint (none) -> Capacitor_SMD:C_0402_1005Metric
- U34, U35, U36, U37: footprint (none) -> Package_SO:SOIC-16_3.9x9.9mm_P1.27mm
Connections:
- net E12: now also U37.9 (C4)
- net GND: now also U34.7 (C0)
