File: Tree01.kicad_sch (KiCad schematic)
At the start: 6 parts, among them U28 74LS283, U29 74LS283, U30 74LS283

Commit message: Fixed ERC issues and applied Footprints
Parts:
- C26, C27, C28: footprint (none) -> Capacitor_SMD:C_0402_1005Metric
- U28, U29, U30: footprint (none) -> Package_SO:SOIC-16_3.9x9.9mm_P1.27mm
Connections:
- net D00: now also U28.4 (S1)
- net D01: now also U28.1 (S2)
- net D02: now also U28.13 (S3)
- net D03: now also U28.10 (S4)
- net GND: now also U28.7 (C0)
